File: axion.sch (EAGLE design)
At the start: 148 parts, among them IC1 3.3V, IC2 5V, Q1 200mA/50V, Q2 12.288Mhz, Q3 200mA/50V, U10 MIC2039, U11 WM8731, U2 Intel Edison, U4 FT232RLSSOP, U6 74HC4050, U7 TPA2005D1DGN, X1 MKDSN1,5/2-5,08, X2 ZX62R-AB-5P, X3 ST-005-G, X4 ZX62R-B-5P

Commit message: Bump the version number
Other:
- note added: "v1.0.0"
- note removed: "v0.9.2"
Changed lines of the file:
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@@
 <plain>
 <text x="194.31" y="-152.4" size="2.1844" layer="94" font="vector">Copyright (c) 2016</text>
-<text x="264.16" y="-139.7" size="2.54" layer="94" font="vector">v0.9.2</text>
+<text x="264.16" y="-139.7" size="2.54" layer="94" font="vector">v1.0.0</text>
 <text x="213.36" y="-136.144" size="2.54" layer="94" font="vector">YMDOC-MXSCH</text>
 <text x="68.58" y="-114.3" size="1.778" layer="91">GAIN=150k/Ｒｉn*2 (2~20)</text>
